Commit message: Fix the robot not moving, and an odometry setting that faked the results
Five more defects found by running the simulation rather than reading it.

1. The robot did not move at all. Both caster spheres and both drive wheels
   bottomed out at exactly z = 0, leaving the load split between them
   numerically indeterminate. ODE resolved the stiff sphere-plane contacts
   first, the drive wheels ended up carrying no normal force, and the robot sat
   still on two mu=0.02 casters while its wheels turned at exactly the
   commanded rate — 3.000 rad/s for a 0.3 m/s command.

   Nothing reported an error. The diff drive plugin loaded, found its joints,
   subscribed to /cmd_vel and drove them correctly; Nav2 planned and commanded
   0.8 m/s; the wheels spun; the robot stayed at x = -12.000 across 4909
   ground-truth samples. Diagnosing it took reading per-link twists out of
   /gazebo/link_states, because every other signal in the system looked healthy.

   Holding the casters 3 mm clear puts the weight on the drive wheels. The
   robot now drives at 0.258 m/s against a 0.3 m/s command and covers 1.5 m in
   6 s. Guarded by test_casters_clear_the_floor.

2. odometry_source was 1, which is WORLD, not ENCODER. The enum in
   gazebo_plugins is ENCODER = 0, WORLD = 1, and this file had 1 with a comment
   asserting it meant ENCODER — so wheel odometry was the simulator's exact
   pose. Every localisation number would have come out flawless while measuring
   nothing, and nothing anywhere would have flagged it.

   Worse, test_config_consistency.py asserted the value was 1 and explained why
   that was correct. The test was confidently enforcing the bug. Both are fixed
   and the test now pins the value to 0 with the enum quoted.

3. The costmap footprint was narrower than the robot. The drive wheels are
   0.05 m wide centred at y = +/-0.25, so they reach +/-0.275, 25 mm proud of
   the chassis on each side. The footprint was set from base_width and so
   understated the robot by exactly the parts that stick out furthest — the
   ones that would clip a racking upright. The footprint is now 0.55 m wide and
   the test computes the requirement from wheel_separation and wheel_width
   rather than trusting base_width.

4. The Nav2 readiness gate was too tight. 60 s tripped on a healthy startup:
   controller_server had configured cleanly with all seven DWB critics loaded
   and was simply mid-activation. Raised to 180 s to match the localisation
   wait, and the diagnostic now covers all nine lifecycle nodes with per-call
   timeouts. A gate that fires on a slow-but-working startup is worse than no
   gate.

5. Docs corrected for the new geometry: inscribed radius 0.275 m,
   circumscribed 0.445 m, residual inflation cost at the boundary 82 rather
   than 76.

176 tests pass, lint clean.

File: src/amr_description/urdf/amr.gazebo.xacro (robot description, xacro)
@@ -40,10 +40,18 @@
       <odometry_frame>odom</odometry_frame>
       <robot_base_frame>base_footprint</robot_base_frame>
-      <!-- ENCODER, not WORLD. WORLD makes the plugin publish Gazebo's exact
-           pose as odometry, which removes every source of drift and turns the
-           localisation evaluation into a measurement of nothing. ENCODER
-           integrates the wheel joints, so the odometry accumulates error the
-           way real encoders do. -->
-      <odometry_source>1</odometry_source>
+      <!-- 0 = ENCODER, 1 = WORLD. Check the enum before changing this.
+           gazebo_plugins' ROS 2 GazeboRosDiffDrive declares
+               enum OdomSource { ENCODER = 0, WORLD = 1 };
+           This file previously said 1 with a comment claiming it meant ENCODER.
+           It does not: 1 publishes Gazebo's exact pose as odometry, which
+           removes every source of drift and turns the whole localisation
+           evaluation into a measurement of nothing — wheel odometry would have
+           come out perfect and the EKF and AMCL would have had nothing to
+           correct. Nothing warns you; the numbers just come out implausibly
+           good.
+           ENCODER integrates the wheel joints, so odometry accumulates error
+           the way real encoders do, including through wheel slip.
+           tests/test_config_consistency.py pins the value to 0. -->
+      <odometry_source>0</odometry_source>
       <publish_odom>true</publish_odom>
       <!-- The EKF owns odom -> base_link. If the plugin also published it there

File: src/amr_description/urdf/amr.urdf.xacro (robot description, xacro)
@@ -29,4 +29,18 @@
   <xacro:property name="caster_radius" value="0.04"/>
   <xacro:property name="caster_mass"   value="0.5"/>
+  <!-- Casters sit this far ABOVE the floor when the drive wheels are on it.
+       3 mm, and it is the difference between a robot that drives and one that
+       does not.
+       Sized so both casters and both wheels bottom out at exactly z = 0 and the
+       load split between them is numerically indeterminate. ODE resolves the
+       stiff sphere-plane point contacts first, lifting the chassis by a
+       hair, and the drive wheels end up carrying no normal force. They then
+       spin at exactly the commanded rate — 3.000 rad/s for 0.3 m/s — while the
+       robot sits still on two mu=0.02 casters. Every plugin reports success and
+       nothing in any log is wrong.
+       Lifting the casters puts the weight on the drive wheels, where it
+       belongs. The robot pitches a fraction of a degree onto whichever caster
+       is loaded, exactly as a real two-wheel-plus-caster AMR does. -->
+  <xacro:property name="caster_clearance" value="0.003"/>
   <!-- Sensor mounting. The 2D LiDAR sits low and forward, at the height that
        sees pallet feet and the underside of a shelf beam. The 3D LiDAR sits on
@@ -125,5 +139,5 @@
       <parent link="base_link"/>
       <child link="${prefix}_caster_link"/>
-      <origin xyz="${x} 0 ${caster_radius - wheel_radius}" rpy="0 0 0"/>
+      <origin xyz="${x} 0 ${caster_radius - wheel_radius + caster_clearance}" rpy="0 0 0"/>
     </joint>
     <gazebo reference="${prefix}_caster_link">
