Commit message: Fix the mission: a person in the aisle closed it at inflation_radius 0.65
The six-waypoint mission now completes. AMCL holds 0.119 m RMSE over 56 m with
zero discontinuities above 0.5 m, and wheel odometry's path length is within 0%
of ground truth, meaning the robot never slipped -- earlier runs over-reported
by 276%, 169%, 56% and 36%, every one of them a robot pinned against something
with its wheels turning.

The cause was geometry, not tuning. A person stands at (8.0, 0.0), dead centre
of a 2.8 m aisle. Inflated by 0.65 from the obstacle and 0.65 from the racking,
the two bands overlapped by 0.15 m and closed the aisle: no zero-cost route past
them existed and NavFn ended runs with "failed to create plan". The robot drove
to within 8 cm of the person, sat rotating for 21 s because DWB hard-rejects any
trajectory entering the inscribed band, threaded the gap by chance, and ended
against the north rack face.

inflation_radius is now 0.47, pinned inside a 5 cm window: above the 0.445
circumscribed radius, below the 0.498 at which a centre-aisle person closes the
lane to less than twice the measured localisation RMSE. cost_scaling_factor
follows from it at 5.8, holding the boundary residual at 82 as before.

The stall also explains a number that looked like a localisation failure and was
not. AMCL held 0.058 m RMSE for the first 53 s, then slid 0.79 m while the robot
stood still with its wheels turning, because odometry reported motion the flat
corridor likelihood could not contradict. Whole-run ATE was 0.476 m. The time
series was actionable; the aggregate pointed at the wrong subsystem.

Also reverted PathDist/PathAlign 44/40 to the 32/32 defaults. They were raised
by argument, made the return to centreline underdamped, and restoring them
changed nothing measurable -- which is what pointed at speed as the constraint.
max_vel_x is 0.45 so the rollout is shorter than the gap being threaded.

The fault-injection harness is rebuilt in the same commit, because running it is
what surfaced the rest. It had never produced a matrix:

* faults.json was written only once the whole schedule had drained, and a fault
  run is expected to abort, so an abort at fault 3 of 5 recorded nothing.
* The sensor dropout was `pkill -STOP -f gzserver`, which suspends the whole
  simulator; under use_sim_time that stops the clock and no node observes a
  dropout at all. It is now a real relay (amr_bringup/scan_relay) that the
  injector tells to stop forwarding, in the LiDAR path only for fault runs so
  the measured localisation figures stay comparable.
* The dropout sat at 120 s behind a kidnap the stack is not designed to survive,
  so it had never once executed.
* All five faults ran in one mission, so each landed on a robot the previous one
  had already broken. Now one fault per run.
* `ros2 topic echo --once` blocks forever on a topic that never appears, which
  made the startup deadline in all three harness scripts unreachable. A test
  now asserts every such call is wrapped in a timeout.

Tests: 198, up from 191. The new ones assert the aisle-lane bound against the
world generator and the fault schedule, so moving a person or retargeting the
block_aisle teleport re-derives the limit rather than silently invalidating it.

File: src/amr_description/urdf/amr.gazebo.xacro (robot description, xacro)
@@ -101,5 +101,5 @@
         <ros>
           <namespace>/</namespace>
-          <remapping>~/out:=scan</remapping>
+          <remapping>~/out:=$(arg scan_topic)</remapping>
         </ros>
         <output_type>sensor_msgs/LaserScan</output_type>

File: src/amr_description/urdf/amr.urdf.xacro (robot description, xacro)
@@ -14,4 +14,10 @@
 <robot name="warehouse_amr" xmlns:xacro="http://www.ros.org/wiki/xacro">
   <xacro:arg name="use_gazebo" default="true"/>
+  <!-- Where the 2D LiDAR publishes. Normally "scan", straight to the stack.
+       The fault-injection run sets this to "scan_raw" and interposes
+       amr_bringup's scan_relay, which can be told to go quiet to simulate a
+       sensor dropout. Keeping it a parameter means every other run is wired
+       exactly as it was measured, with no relay in the path. -->
+  <xacro:arg name="scan_topic" default="scan"/>
   <!-- Body: 0.70 x 0.50 x 0.28 m chassis, 65 kg laden. -->
   <xacro:property name="base_length" value="0.70"/>

Commit message: Migrate the simulation from Gazebo Classic 11 to gz-sim Harmonic on ROS 2 Jazzy
Gazebo Classic reached end of life in January 2025. Jazzy and Harmonic are the
officially paired long-term releases, and Jazzy's ros_gz packages bring
Harmonic with them through the vendor packages.

The world, robot and sensors are kept equivalent: same geometry, 1 ms step,
sensor rates, resolutions, ranges and noise, drive geometry and limits.
gz-sim systems replace the gazebo_ros plugins (DiffDrive, gpu_lidar x2, Imu,
JointStatePublisher, OdometryPublisher for ground truth) and ros_gz_bridge
carries every topic, plus the set_pose service the fault injector uses.

Things the migration had to deal with, each pinned by a config test:
- gz.msgs.Odometry has no covariance; odom_covariance restores the values the
  Classic plugin advertised so the EKF does not trust the wheels absolutely.
- set_pose does not move a static model's collision or visual, so faults move
  a dynamic fault_pallet parked outside the building.
- Jazzy Nav2: no built-in BT plugin list, scoped plugin names, plural
  progress checker key, local_frame on the behaviour server, BT.CPP v4.
- RotateToGoal reads FollowPath.xy_goal_tolerance, not a RotateToGoal key, so
  the old setting was ignored and the robot stopped 0.24 m short of goals.
- The fault schedule clock now starts when a navigation goal executes, and
  the mission runner waits for bt_navigator to be active, not merely present.

File: src/amr_description/urdf/amr.gazebo.xacro (robot description, xacro)
@@ -1,6 +1,12 @@
 <?xml version="1.0"?>
 <!--
-  Gazebo plugins: differential drive, 2D LiDAR, 3D LiDAR, IMU, and a ground
-  truth pose publisher.
+  Gazebo (gz-sim 8, Harmonic) systems and sensors: differential drive, 2D LiDAR,
+  3D LiDAR, IMU, wheel joint states and a ground truth pose publisher.
+  Migrated from Gazebo Classic 11, which reached end of life in January 2025.
+  Every sensor keeps its Classic rate, resolution, range and noise, and the
+  drive keeps its geometry and limits, so the robot the stack sees is the same
+  robot. What changed is the transport: gz-sim systems publish on gz-transport
+  topics and ros_gz_bridge (amr_bringup/config/gz_bridge.yaml) carries them into
+  ROS. Nothing in this file talks to ROS directly.
   Sensor noise is set deliberately, not left at zero. A noiseless simulation
   produces localisation numbers that cannot be reproduced on hardware and that
@@ -11,70 +17,78 @@
 -->
 <robot xmlns:xacro="http://www.ros.org/wiki/xacro">
-  <gazebo reference="base_link">
-    <material>Gazebo/Grey</material>
-  </gazebo>
   <!-- ==================================================================== -->
   <!-- Differential drive                                                    -->
   <!-- ==================================================================== -->
   <gazebo>
-    <plugin name="diff_drive" filename="libgazebo_ros_diff_drive.so">
-      <ros>
-        <namespace>/</namespace>
-        <remapping>cmd_vel:=cmd_vel</remapping>
-        <remapping>odom:=odom</remapping>
-      </ros>
-      <update_rate>50</update_rate>
+    <plugin filename="gz-sim-diff-drive-system" name="gz::sim::systems::DiffDrive">
       <left_joint>left_wheel_joint</left_joint>
       <right_joint>right_wheel_joint</right_joint>
       <wheel_separation>0.50</wheel_separation>
-      <wheel_diameter>0.20</wheel_diameter>
-      <!-- Torque to accelerate 65 kg at 1.0 m/s^2 is 32.5 N per wheel, or
-           3.25 Nm at a 0.10 m radius. 25 Nm leaves ample margin for the ramp
-           onto a dock and for pushing through a floor seam. -->
-      <max_wheel_torque>25.0</max_wheel_torque>
-      <!-- rad/s^2, NOT m/s^2. At a 0.10 m wheel radius this is 1.0 m/s^2 at the
-           contact patch, which is what acc_lim_x in nav2_params.yaml is set to.
-           These two numbers must agree: a DWB that plans deceleration the base
-           cannot deliver will overshoot every goal and clip every corner. -->
-      <max_wheel_acceleration>10.0</max_wheel_acceleration>
-      <odometry_frame>odom</odometry_frame>
-      <robot_base_frame>base_footprint</robot_base_frame>
-      <!-- 0 = ENCODER, 1 = WORLD. Check the enum before changing this.
-           gazebo_plugins' ROS 2 GazeboRosDiffDrive declares
-               enum OdomSource { ENCODER = 0, WORLD = 1 };
-           This file previously said 1 with a comment claiming it meant ENCODER.
-           It does not: 1 publishes Gazebo's exact pose as odometry, which
-           removes every source of drift and turns the whole localisation
-           evaluation into a measurement of nothing — wheel odometry would have
-           come out perfect and the EKF and AMCL would have had nothing to
-           correct. Nothing warns you; the numbers just come out implausibly
-           good.
-           ENCODER integrates the wheel joints, so odometry accumulates error
-           the way real encoders do, including through wheel slip.
-           tests/test_config_consistency.py pins the value to 0. -->
-      <odometry_source>0</odometry_source>
-      <publish_odom>true</publish_odom>
-      <!-- The EKF owns odom -> base_link. If the plugin also published it there
-           would be two publishers on one transform and the tree would flip
-           between them. -->
-      <publish_odom_tf>false</publish_odom_tf>
-      <publish_wheel_tf>true</publish_wheel_tf>
-      <!-- Covariance the plugin advertises on /odom. The EKF reads these, so
-           they have to be honest rather than optimistic. -->
-      <covariance_x>0.001</covariance_x>
-      <covariance_y>0.001</covariance_y>
-      <covariance_yaw>0.01</covariance_yaw>
+      <wheel_radius>0.10</wheel_radius>
+      <!-- Absolute topic names, so the bridge does not need to know the model
+           name. cmd_vel arrives from Nav2's velocity smoother. -->
+      <topic>/cmd_vel</topic>
+      <!-- Odometry is integrated from the wheel joint positions, the way real
+           encoders work, including through wheel slip. gz-sim's DiffDrive has
+           no "world" source at all, which retires the Classic trap where
+           odometry_source 1 silently published ground truth as odometry.
+           It publishes on odom_raw rather than odom because gz.msgs.Odometry
+           carries no covariance, so the bridged message has an all-zero
+           matrix. robot_localization clamps a zero variance to 1e-9 and would
+           then trust the wheels absolutely. amr_bringup's odom_covariance node
+           stamps the covariance the Classic plugin advertised and republishes
+           on /odom. -->
+      <odom_topic>/odom_raw</odom_topic>
+      <odom_publish_frequency>50</odom_publish_frequency>
+      <frame_id>odom</frame_id>
+      <child_frame_id>base_footprint</child_frame_id>
+      <!-- The EKF owns odom -> base_footprint. The system always publishes a
+           transform, so it goes to a gz topic that nothing bridges; the effect
+           is the Classic publish_odom_tf false. -->
+      <tf_topic>/model/warehouse_amr/tf_unused</tf_topic>
+      <!-- 1.0 m/s^2 at the contact patch, which is what acc_lim_x in
+           nav2_params.yaml is set to. These two numbers must agree: a DWB that
+           plans deceleration the base cannot deliver will overshoot every goal
+           and clip every corner. Classic expressed this as 10 rad/s^2 of wheel
+           acceleration at a 0.10 m radius, the same value.
+           Angular: each wheel at 1.0 m/s^2 in opposite directions over a
+           0.50 m track is 2 x 1.0 / 0.50 = 4.0 rad/s^2, which is the limit the
+           Classic wheel-acceleration cap imposed on a spin. -->
+      <max_linear_acceleration>1.0</max_linear_acceleration>
+      <min_linear_acceleration>-1.0</min_linear_acceleration>
+      <max_angular_acceleration>4.0</max_angular_acceleration>
+      <min_angular_acceleration>-4.0</min_angular_acceleration>
     </plugin>
+    <!-- Wheel joint angles, so robot_state_publisher can place the wheel
+         links. Classic's diff drive did this with publish_wheel_tf. Without
+         update_rate it publishes on every 1 ms physics step, and the bridge
+         and robot_state_publisher spend a core forwarding wheel angles. -->
+    <plugin filename="gz-sim-joint-state-publisher-system"
+            name="gz::sim::systems::JointStatePublisher">
+      <topic>/joint_states</topic>
+      <update_rate>50</update_rate>
+      <joint_name>left_wheel_joint</joint_name>
+      <joint_name>right_wheel_joint</joint_name>
+    </plugin>
   </gazebo>
   <!-- ==================================================================== -->
   <!-- 2D LiDAR: AMCL, Cartographer, scan odometry, Nav2 obstacle layer      -->
+  <!--                                                                       -->
+  <!-- gpu_lidar is the only LiDAR gz-sim has: it is rendered by ogre2, so a  -->
+  <!-- headless run needs a GL implementation. In CI and Docker that is      -->
+  <!-- Mesa's llvmpipe on the CPU; see docs/simulation.md.                   -->
   <!-- ==================================================================== -->
   <gazebo reference="lidar_2d_link">
-    <material>Gazebo/Blue</material>
-    <sensor name="lidar_2d" type="ray">
+    <sensor name="lidar_2d" type="gpu_lidar">
       <pose>0 0 0 0 0 0</pose>
+      <!-- Without this the message is stamped with the scoped gz frame name,
+           which is not in the TF tree, because sdformat folds fixed-joint
+           links into their parent. -->
+      <gz_frame_id>lidar_2d_link</gz_frame_id>
+      <topic>/$(arg scan_topic)</topic>
+      <always_on>true</always_on>
       <visualize>false</visualize>
       <update_rate>10.0</update_rate>
-      <ray>
+      <lidar>
         <scan>
           <horizontal>
@@ -86,4 +100,10 @@
             <max_angle>3.14159</max_angle>
           </horizontal>
+          <vertical>
+            <samples>1</samples>
+            <resolution>1</resolution>
+            <min_angle>0</min_angle>
+            <max_angle>0</max_angle>
+          </vertical>
         </scan>
         <range>
@@ -97,13 +117,5 @@
           <stddev>0.01</stddev>
         </noise>
-      </ray>
-      <plugin name="lidar_2d_controller" filename="libgazebo_ros_ray_sensor.so">
-        <ros>
-          <namespace>/</namespace>
-          <remapping>~/out:=$(arg scan_topic)</remapping>
-        </ros>
-        <output_type>sensor_msgs/LaserScan</output_type>
-        <frame_name>lidar_2d_link</frame_name>
-      </plugin>
+      </lidar>
     </sensor>
   </gazebo>
@@ -112,10 +124,14 @@
   <!-- ==================================================================== -->
   <gazebo reference="lidar_3d_link">
-    <material>Gazebo/Blue</material>
-    <sensor name="lidar_3d" type="ray">
+    <sensor name="lidar_3d" type="gpu_lidar">
       <pose>0 0 0 0 0 0</pose>
+      <gz_frame_id>lidar_3d_link</gz_frame_id>
+      <!-- gpu_lidar publishes a LaserScan on <topic> and the point cloud on
+           <topic>/points; the bridge carries only the cloud. -->
+      <topic>/lidar_3d</topic>
+      <always_on>true</always_on>
       <visualize>false</visualize>
       <update_rate>10.0</update_rate>
-      <ray>
+      <lidar>
         <scan>
           <horizontal>
@@ -148,13 +164,5 @@
           <stddev>0.01</stddev>
         </noise>
-      </ray>
-      <plugin name="lidar_3d_controller" filename="libgazebo_ros_ray_sensor.so">
-        <ros>
-          <namespace>/</namespace>
-          <remapping>~/out:=lidar_3d/points</remapping>
-        </ros>
-        <output_type>sensor_msgs/PointCloud2</output_type>
-        <frame_name>lidar_3d_link</frame_name>
-      </plugin>
+      </lidar>
     </sensor>
   </gazebo>
@@ -164,4 +172,6 @@
   <gazebo reference="imu_link">
     <sensor name="imu" type="imu">
+      <gz_frame_id>imu_link</gz_frame_id>
+      <topic>/imu/data</topic>
       <always_on>true</always_on>
       <update_rate>100</update_rate>
@@ -188,12 +198,4 @@
         </linear_acceleration>
       </imu>
-      <plugin name="imu_controller" filename="libgazebo_ros_imu_sensor.so">
-        <ros>
-          <namespace>/</namespace>
-          <remapping>~/out:=imu/data</remapping>
-        </ros>
-        <frame_name>imu_link</frame_name>
-        <initial_orientation_as_reference>false</initial_orientation_as_reference>
-      </plugin>
     </sensor>
   </gazebo>
@@ -205,17 +207,17 @@
   <!-- ONLY consumer of it. Nothing in the navigation or localisation stack    -->
   <!-- subscribes to this topic; if anything did, the evaluation would be      -->
-  <!-- measuring the simulator against itself. analysis/localisation_error.py  -->
-  <!-- asserts that the recorded run contains no such subscriber.              -->
+  <!-- measuring the simulator against itself. pose_logger checks that at      -->
+  <!-- runtime. Replaces Classic's gazebo_ros_p3d.                             -->
   <!-- ==================================================================== -->
   <gazebo>
-    <plugin name="ground_truth" filename="libgazebo_ros_p3d.so">
-      <ros>
-        <namespace>/</namespace>
-        <remapping>odom:=ground_truth/pose</remapping>
-      </ros>
-      <frame_name>world</frame_name>
-      <body_name>base_footprint</body_name>
-      <update_rate>50.0</update_rate>
-      <gaussian_noise>0.0</gaussian_noise>
+    <plugin filename="gz-sim-odometry-publisher-system"
+            name="gz::sim::systems::OdometryPublisher">
+      <odom_frame>world</odom_frame>
+      <robot_base_frame>base_footprint</robot_base_frame>
+      <odom_topic>/ground_truth/pose</odom_topic>
+      <odom_covariance_topic>/ground_truth/pose_cov_unused</odom_covariance_topic>
+      <tf_topic>/ground_truth/tf_unused</tf_topic>
+      <odom_publish_frequency>50</odom_publish_frequency>
+      <dimensions>3</dimensions>
     </plugin>
   </gazebo>

File: src/amr_description/urdf/amr.urdf.xacro (robot description, xacro)
@@ -39,5 +39,5 @@
        does not.
        Sized so both casters and both wheels bottom out at exactly z = 0 and the
-       load split between them is numerically indeterminate. ODE resolves the
+       load split between them is numerically indeterminate. the contact solver resolves the
        stiff sphere-plane point contacts first, lifting the chassis by a
        hair, and the drive wheels end up carrying no normal force. They then
@@ -116,4 +116,11 @@
       <origin xyz="0 ${reflect * wheel_separation / 2.0} 0" rpy="0 0 0"/>
       <axis xyz="0 1 0"/>
+      <!-- 25 Nm, the Classic plugin's max_wheel_torque. Torque to accelerate
+           65 kg at 1.0 m/s^2 is 32.5 N per wheel, or 3.25 Nm at a 0.10 m
+           radius, so this leaves ample margin for a ramp or a floor seam.
+           gz-sim's DiffDrive commands wheel velocity and DART holds it with at
+           most this effort, so the limit lives on the joint now. velocity is
+           required by the URDF schema; 30 rad/s (3 m/s) is never reached. -->
+      <limit effort="25.0" velocity="30.0"/>
       <dynamics damping="0.05" friction="0.1"/>
     </joint>
@@ -126,5 +133,4 @@
       <kp>1000000.0</kp>
       <kd>100.0</kd>
-      <material>Gazebo/DarkGrey</material>
     </gazebo>
   </xacro:macro>
@@ -150,5 +156,4 @@
       <mu1>0.02</mu1>
       <mu2>0.02</mu2>
-      <material>Gazebo/DarkGrey</material>
     </gazebo>
   </xacro:macro>
