Commit message: Give the wheels a thin contact disc: DART was turning the robot 11% too far
DART puts a cylinder's floor contacts at its rim edges. With the 50 mm tyre
as the wheel collision the inner edges carried the load, so the effective
track was 0.45 m against the 0.50 m DiffDrive integrates with. One commanded
turn in place came out as 397 degrees by ground truth and 358 by wheel
odometry, and the full mission's wheel-odometry heading error reached 85
degrees RMS. A 4 mm collision disc in the tyre's plane brings it to 361
against 358; the visual and the lateral envelope are unchanged.

Also score the EKF in make eval, as the open-loop harness already did.

File: src/amr_description/urdf/amr.urdf.xacro (robot description, xacro)
@@ -31,4 +31,15 @@
   <xacro:property name="wheel_radius"    value="0.10"/>
   <xacro:property name="wheel_width"     value="0.05"/>
+  <!-- The wheel's COLLISION is a 4 mm disc, not the 50 mm tyre the visual
+       shows. DART puts a cylinder's contacts with the floor at its rim edges,
+       and with a 50 mm tyre the inner edges carry the load, so the effective
+       track was 0.45 m against the 0.50 m DiffDrive integrates with. Measured
+       on gz-sim: commanded one full turn in place, wheel odometry reported
+       358 degrees while ground truth turned 397, an 11% overspin that wrecked
+       wheel-odometry heading on every in-place turn. With a 4 mm contact
+       width the track is within 1% (358 against 361). Classic's ODE did not
+       do this. The lateral envelope is unchanged: the disc sits in the same
+       plane as the tyre and inside the chassis footprint. -->
+  <xacro:property name="wheel_contact_width" value="0.004"/>
   <xacro:property name="wheel_mass"      value="2.0"/>
   <xacro:property name="wheel_separation" value="0.50"/>
@@ -107,5 +118,5 @@
       <collision>
         <origin xyz="0 0 0" rpy="${pi/2.0} 0 0"/>
-        <geometry><cylinder radius="${wheel_radius}" length="${wheel_width}"/></geometry>
+        <geometry><cylinder radius="${wheel_radius}" length="${wheel_contact_width}"/></geometry>
       </collision>
       <xacro:cylinder_inertia m="${wheel_mass}" r="${wheel_radius}" h="${wheel_width}"/>
